File: TP1/Tomi/Fuente de alimentación.kicad_pcb (KiCad board)
At the start: 2 copper layers, 58.5 x 32.5 mm, 17 parts, among them J1 Barrel_Jack_Switch, J2 Conn_01x04_Pin, J3 Conn_01x04_Pin, J4 Conn_01x02_Pin, J5 Conn_01x01_Pin, J6 Conn_01x01_Pin, U1 L7805, U2 AZ1117-3.3

Commit message: actualizo pcb
Parts:
- GND IN: renamed from J6
- VCC IN: renamed from J5
Other:
- board size 58.5 x 32.5 mm -> 57 x 33.5 mm
- board text added: "3.3V"
- board text added: "5V"
- board text added: "GND"
- board text added: "VCC"
Changed lines of the file:
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@@
 		(descr "Through hole straight pin header, 1x01, 2.54mm pitch, single row")
 		(tags "Through hole pin header THT 1x01 2.54mm single row")
-		(property "Reference" "J5"
+		(property "Reference" "VCC IN"
 			(at 0 -2.38 0)
 			(layer "F.SilkS")
 			(effects
 				(font
-					(size 1 1)
-					(thickness 0.15)
+					(size 0.8 0.8)
+					(thickness 0.1)
 				)
 			)
@@
 		(descr "Through hole straight pin header, 1x01, 2.54mm pitch, single row")
 		(tags "Through hole pin header THT 1x01 2.54mm single row")
-		(property "Reference" "J6"
+		(property "Reference" "GND IN"
 			(at 0 -2.38 0)
 			(layer "F.SilkS")
@@
 	)
 	(gr_rect
-		(start 108 64)
-		(end 166.5 96.5)
+		(start 108 63)
+		(end 165 96.5)
 		(stroke
 			(width 0.05)
@@
 		)
 	)
+	(gr_text "5V"
+		(at 137.5 70.5 90)
+		(layer "F.SilkS")
+		(effects
+			(font
+				(size 0.7 0.7)
+				(thickness 0.1)
+			)
+		)
+	)
+	(gr_text "5V"
+		(at 164 78 90)
+		(layer "F.SilkS")
+		(effects
+			(font
+				(size 0.7 0.7)
+				(thickness 0.1)
+			)
+		)
+	)
+	(gr_text "GND"
+		(at 164 83.5 90)
+		(layer "F.SilkS")
+		(effects
+			(font
+				(size 0.7 0.7)
+				(thickness 0.1)
+			)
+		)
+	)
+	(gr_text "GND"
+		(at 145.5 89 0)
+		(layer "F.SilkS")
+		(effects
+			(font
+				(size 0.7 0.7)
+				(thickness 0.1)
+			)
+		)
+	)
+	(gr_text "5V"
+		(at 140 89 0)
+		(layer "F.SilkS")
+		(effects
+			(font
+				(size 0.7 0.7)
+				(thickness 0.1)
+			)
+		)
+	)
+	(gr_text "3.3V"
+		(at 164 81 90)
+		(layer "F.SilkS")
+		(effects
+			(font
+				(size 0.7 0.7)
+				(thickness 0.1)
+			)
+		)
+	)
+	(gr_text "3.3V"
+		(at 142.5 89 0)
+		(layer "F.SilkS")
+		(effects
+			(font
+				(size 0.7 0.7)
+				(thickness 0.1)
+			)
+		)
+	)
+	(gr_text "GND"
+		(at 137.5 67.5 90)
+		(layer "F.SilkS")
+		(effects
+			(font
+				(size 0.7 0.7)
+				(thickness 0.1)
+			)
+		)
+	)
+	(gr_text "VCC"
+		(at 164 75.5 90)
+		(layer "F.SilkS")
+		(effects
+			(font
+				(size 0.7 0.7)
+				(thickness 0.1)
+			)
+		)
+	)
+	(gr_text "VCC"
+		(at 137.5 89 0)
+		(layer "F.SilkS")
+		(effects
+			(font
+				(size 0.7 0.7)
+				(thickness 0.1)
+			)
+		)
+	)
 	(via
 		(at 161.5 68)
@@
 		(hatch edge 0.5)
 		(connect_pads
-			(clearance 1)
+			(clearance 0.75)
 		)
 		(min_thickness 0.25)
@@
 		(fill yes
 			(thermal_gap 0.5)
-			(thermal_bridge_width 0.5)
+			(thermal_bridge_width 0.75)
 			(island_removal_mode 1)
 			(island_area_min 10)
@@
 		(polygon
 			(pts
-				(xy 109 64.5) (xy 109 94.5) (xy 165.5 95) (xy 165 64.5)
+				(xy 109 64) (xy 164 64) (xy 164 95.5) (xy 109 95.5)
 			)
 		)
